File: ELECTRONICS/6502_SBC.sch (KiCad schematic (older format))
At the start: 19 parts, among them J1 Conn_01x06_Female, J2 Conn_02x20_Odd_Even, SW1 SW_Push, U1 7400, U2 W65C02S, U3 71256SA, U4 71256SA, U5 PIC18F15Q41-IP

Commit message: Add files via upload
Parts:
- U3: value 71256SA -> 62256
- U4: value 71256SA -> 28C64
Changed lines of the file:
@@
 P 4700 2450
 F 0 "U3" H 4700 3750 50  0000 C CNN
-F 1 "71256SA" H 4700 3650 50  0000 C CNN
+F 1 "62256" H 4700 3650 50  0000 C CNN
 F 2 "Package_DIP:DIP-28_W15.24mm_Socket_LongPads" H 4700 2450 50  0001 C CNN
 F 3 "" H 4700 2450 50  0001 C CNN
@@
 P 7300 2450
 F 0 "U4" H 7300 3750 50  0000 C CNN
-F 1 "71256SA" H 7300 3650 50  0000 C CNN
+F 1 "28C64" H 7300 3650 50  0000 C CNN
 F 2 "Package_DIP:DIP-28_W15.24mm_Socket_LongPads" H 7300 2450 50  0001 C CNN
 F 3 "" H 7300 2450 50  0001 C CNN
